Commit message: attempting rewrite of xacro output

File: robot_calibration_tests/urdf/argo_tracker_with_error.urdf (robot description, URDF)
Before this commit: robot taurob_tracker, 32 links, 31 joints
Links:
- removed link chilitag4_background_link
- removed link chilitag5_background_link
- removed link chilitag7_background_link
- added link arm_rgbd_cam_rgb_frame
- added link arm_rgbd_cam_rgb_optical_frame
- link chilitag4_link: mass 0.01 -> None; geometry 
- link chilitag5_link: mass 0.01 -> None; geometry 
- link chilitag7_link: mass 0.01 -> None; geometry 
- link flipper_link_1: mass 1.0 -> 10.0
- link spin_lidar_lidar_mount_link: geometry collision cylinder length=0.145 radius=0.1
- link structure_addons_link: geometry collision box size=0.135 0.32 0.08; collision box size=0.17 0.135 0.2
Joints:
- removed joint chilitag4_background_joint
- removed joint chilitag5_background_joint
- removed joint chilitag7_background_joint
- added joint arm_rgbd_cam_rgb_joint: type fixed, parent arm_rgbd_cam_link, child arm_rgbd_cam_rgb_frame, origin xyz=0 0 0 rpy=0 0 0
- added joint arm_rgbd_cam_rgb_optical_joint: type fixed, parent arm_rgbd_cam_rgb_frame, child arm_rgbd_cam_rgb_optical_frame, origin xyz=0 0 0 rpy=-1.571 0.000 -1.571
- joint arm_joint_0: origin xyz=0.12 0 0.24238 rpy=0 0 1.6707963268 -> xyz=0.12 0 0.24238 rpy=0 0 1.5707963268
- joint arm_joint_1: origin xyz=-0.067 0.0 0.06 rpy=0.1 0 0 -> xyz=-0.067 0.0 0.06 rpy=0 0 0
- joint arm_joint_2: origin xyz=0.022 0.551 0.0 rpy= 0.1 0 0 -> xyz=0.022 0.551 0.0 rpy=0 0 0
- joint arm_rgbd_cam_joint: origin xyz=0.136 0.0413 0.0464 rpy=1.5707963268 0 0 -> xyz=0.136 0.0413 0.0464 rpy=1.6707963268 0.1 0.1
- joint arm_zoom_cam_optical_joint: origin xyz=0.003 0.002 0.001 rpy=-1.5807963268 0.01 -1.5807963268 -> xyz=0 0 0 rpy=-1.5707963268 0.0 -1.5707963268
- joint chilitag5_joint: origin xyz=-0.18 -0.05 0 rpy=0 0 0 -> xyz=-0.18 -0.05 0.0 rpy=0 0 0
- joint chilitag7_joint: origin xyz=-0.285 -0.15 0 rpy=0 0 0 -> xyz=-0.285 -0.15 0.0 rpy=0 0 0
- joint chilitag_base_joint: origin xyz=-0.07 0.001 0.001 rpy=0.05 0.04 0.03 -> xyz=-0.068 -0.0 0.001 rpy=0 0 0
- joint flipper_joint_1: limit lower=-0.872664625997 upper=0.523598775598 effort=10000 velocity=1.91986217719 -> lower=-0.872664625997 upper=0.523598775598 effort=10000 velocity=0.523598775598
- joint sensor_head_pitch_joint: origin xyz=0.105 -0.435 -0.013 rpy= 0.1 0 0 -> xyz=0.105 -0.435 -0.013 rpy=0.0 0 0
- joint sensor_head_yaw_joint: origin xyz=0.0405  0.052 0.0655 rpy=0 0 -1.4707963268 -> xyz=0.0405  0.052 0.0655 rpy=0 0 -1.5707963268
